File: car_control/car_control.kicad_pcb (KiCad board)
At the start: 2 copper layers, 179.7 x 76.2 mm, 30 parts, among them J1 Screw_Terminal_01x02, J2 Conn_01x03, J3 Conn_01x03, J4 Screw_Terminal_01x02, J5 Conn_01x06, Q1 IRF540N, Q2 2N3904, SW1 SW_SPST, SW2 SW_Push, U1 TCRT5000

Commit message: diagrams
Parts:
- added REF**: car_as, car_as:car_as, F.Cu at (107.4, 5.71)
Changed lines of the file:
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@@
+    )
+  )
+  (footprint "car_as:car_as" (layer "F.Cu")
+    (at 107.443 5.713)
+    (fp_text reference "REF**" (at 30.48 32.56 unlocked) (layer "F.SilkS")
+        (effects (font (size 1 1) (thickness 0.1)))
+    )
+    (fp_text value "car_as" (at 30.48 34.06 unlocked) (layer "F.Fab")
+        (effects (font (size 1 1) (thickness 0.15)))
+    )
+    (fp_text user "${REFERENCE}" (at 30.48 35.56 unlocked) (layer "F.Fab")
+        (effects (font (size 1 1) (thickness 0.15)))
+    )
+    (fp_line (start 22.86 38.1) (end 139.7 38.1)
+      (stroke (width 0.1) (type default)) (layer "F.SilkS"))
+    (fp_line (start 22.86 127) (end 22.86 38.1)
+      (stroke (width 0.1) (type default)) (layer "F.SilkS"))
+    (fp_line (start 139.7 38.1) (end 139.7 127)
+      (stroke (width 0.1) (type default)) (layer "F.SilkS"))
+    (fp_line (start 139.7 127) (end 22.86 127)
+      (stroke (width 0.1) (type default)) (layer "F.SilkS"))
+    (pad "" np_thru_hole circle (at 38.735 48.006) (size 3.81 3.81) (drill 3.81) (layers "F&B.Cu" "*.Mask"))
+    (pad "" np_thru_hole circle (at 38.735 116.586) (size 3.81 3.81) (drill 3.81) (layers "F&B.Cu" "*.Mask"))
+    (pad "" np_thru_hole circle (at 126.365 82.296) (size 3.81 3.81) (drill 3.81) (layers "F&B.Cu" "*.Mask"))
+    (model "/home/hazen/work/epic-car-control/mech/car_as_footprint.wrl"
+      (offset (xyz 64.135 -82.55 -24.765))
+      (scale (xyz 10 10 10))
+      (rotate (xyz 0 0 0))
     )
   )
