File: car_control/car_control.kicad_sch (KiCad schematic)
At the start: 31 parts, among them J1 Screw_Terminal_01x02, J2 Conn_01x03, J3 Conn_01x03, J4 Screw_Terminal_01x02, J5 Conn_01x06, Q1 IRF540N, Q2 2N3904, SW1 SW_SPST, SW2 SW_Push, U1 TCRT5000

Commit message: add cherry switch, change pwr sw to header, reroute
Parts:
- SW1: footprint mini_slide_switch:OS102011MA1QN1 -> Connector_PinHeader_2.54mm:PinHeader_1x02_P2.54mm_Vertical
- SW2: footprint my_pushbutton:sw_push_6.2x6.2mm_p5 -> my_cherry:SW_Cherry_MX_1.00u_PCB
Changed lines of the file:
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@@
       (effects (font (size 1.27 1.27)))
     )
-    (property "Footprint" "my_pushbutton:sw_push_6.2x6.2mm_p5" (at 57.15 95.25 0)
+    (property "Footprint" "my_cherry:SW_Cherry_MX_1.00u_PCB" (at 57.15 95.25 0)
       (effects (font (size 1.27 1.27)) hide)
     )
@@
       (effects (font (size 1.27 1.27)))
     )
-    (property "Footprint" "mini_slide_switch:OS102011MA1QN1" (at 58.42 46.99 0)
+    (property "Footprint" "Connector_PinHeader_2.54mm:PinHeader_1x02_P2.54mm_Vertical" (at 58.42 46.99 0)
       (effects (font (size 1.27 1.27)) hide)
     )

Commit message: Rev 1 as built
Parts:
- H1, H2, H3, N2: CatNo (none) -> DNP
- J1, J4: CatNo A122765-ND -> Amazon
- Q2: CatNo (none) -> Amazon
- R1, R2, R3, R4, R5, R6, R7: CatNo (none) -> EDF
- SW1: CatNo CKN9559-ND -> Stock
Changed lines of the file:
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@@
+      (effects (font (size 1.27 1.27)) hide)
+    )
+    (property "CatNo" "EDF" (at 154.94 97.79 0)
       (effects (font (size 1.27 1.27)) hide)
     )
@@
       (effects (font (size 1.27 1.27)) hide)
     )
-    (property "CatNo" "A122765-ND" (at 161.29 53.34 0)
+    (property "CatNo" "Amazon" (at 161.29 53.34 0)
       (effects (font (size 1.27 1.27)) hide)
     )
@@
       (effects (font (size 1.27 1.27)) hide)
     )
+    (property "CatNo" "DNP" (at 45.72 176.53 0)
+      (effects (font (size 1.27 1.27)) hide)
+    )
     (instances
       (project "car_control"
@@
       (effects (font (size 1.27 1.27)) hide)
     )
+    (property "CatNo" "DNP" (at 44.45 129.54 0)
+      (effects (font (size 1.27 1.27)) hide)
+    )
     (instances
       (project "car_control"
@@
     )
     (property "Datasheet" "~" (at 205.74 91.44 0)
+      (effects (font (size 1.27 1.27)) hide)
+    )
+    (property "CatNo" "EDF" (at 205.74 91.44 0)
       (effects (font (size 1.27 1.27)) hide)
     )
@@
       (effects (font (size 1.27 1.27)) (justify left) hide)
     )
+    (property "CatNo" "Amazon" (at 83.82 161.29 0)
+      (effects (font (size 1.27 1.27)) hide)
+    )
     (pin "1")
     (pin "2")
@@
       (effects (font (size 1.27 1.27)) hide)
     )
+    (property "CatNo" "EDF" (at 154.94 120.65 0)
+      (effects (font (size 1.27 1.27)) hide)
+    )
     (pin "1")
     (pin "2")
@@
     )
     (property "Datasheet" "~" (at 154.94 113.03 0)
+      (effects (font (size 1.27 1.27)) hide)
+    )
+    (property "CatNo" "EDF" (at 154.94 113.03 0)
       (effects (font (size 1.27 1.27)) hide)
     )
@@
       (effects (font (size 1.27 1.27)) hide)
     )
+    (property "CatNo" "EDF" (at 205.74 86.36 0)
+      (effects (font (size 1.27 1.27)) hide)
+    )
     (pin "1")
     (pin "2")
@@
       (effects (font (size 1.27 1.27)) hide)
     )
-    (property "CatNo" "A122765-ND" (at 38.1 58.42 0)
+    (property "CatNo" "Amazon" (at 38.1 58.42 0)
       (effects (font (size 1.27 1.27)))
     )
@@
       (effects (font (size 1.27 1.27)) hide)
     )
+    (property "CatNo" "DNP" (at 44.45 135.89 0)
+      (effects (font (size 1.27 1.27)) hide)
+    )
     (instances
       (project "car_control"
@@
     )
     (property "Datasheet" "~" (at 44.45 142.24 0)
+      (effects (font (size 1.27 1.27)) hide)
+    )
+    (property "CatNo" "DNP" (at 44.45 142.24 0)
       (effects (font (size 1.27 1.27)) hide)
     )
@@
       (effects (font (size 1.27 1.27)) hide)
     )
+    (property "CatNo" "EDF" (at 72.39 161.29 0)
+      (effects (font (size 1.27 1.27)) hide)
+    )
     (pin "1")
     (pin "2")
@@
       (effects (font (size 1.27 1.27)) hide)
     )
+    (property "CatNo" "EDF" (at 154.94 105.41 0)
+      (effects (font (size 1.27 1.27)) hide)
+    )
     (pin "1")
     (pin "2")
@@
       (effects (font (size 1.27 1.27)) hide)
     )
-    (property "CatNo" "CKN9559-ND" (at 58.42 40.64 0)
-      (effects (font (size 1.27 1.27)))
-    )
+    (property "CatNo" "Stock" (at 58.42 40.64 0)
+      (effects (font (size 1.27 1.27)))
+    )

Commit message: Version 9 with EEPROM sensor limits fixed
Parts:
- R1: value 150 -> 120
- R2: value 240 -> 1.8k
- R3, R4: value 200 -> 220

Commit message: update doco for 2025
Other:
- note added: "Boston University EPIC"
- note added: "Model car control electronics"
Changed lines of the file:
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@@
+		)
+	)
+	(text "Model car control electronics"
+		(exclude_from_sim no)
+		(at 180.594 177.8 0)
+		(effects
+			(font
+				(size 3.175 3.175)
+			)
+			(justify left)
 		)
 	)
@@
 		)
 	)
+	(text "Boston University EPIC"
+		(exclude_from_sim no)
+		(at 223.012 171.196 0)
+		(effects
+			(font
+				(size 5.08 5.08)
+			)
+		)
+	)
